Commit message: Update URDF visual meshes.

File: abb_irb1200_support/urdf/irb1200_7_70_macro.xacro (robot description, xacro)
@@ -14,5 +14,6 @@
       <visual name="visual">
         <geometry>
-          <mesh filename="package://abb_irb1200_support/meshes/irb1200_7_70/visual/base_link.stl" scale="0.001 0.001 0.001" />
+	  <!-- reference irb1200_5_90 package since mesh is shared-->
+          <mesh filename="package://abb_irb1200_support/meshes/irb1200_5_90/visual/base_link.dae" scale="0.001 0.001 0.001" />
         </geometry>
         <material name="graphite_white">
@@ -30,5 +31,6 @@
       <visual name="visual">
         <geometry>
-          <mesh filename="package://abb_irb1200_support/meshes/irb1200_7_70/visual/link_1.stl" scale="0.001 0.001 0.001" />
+	  <!-- reference irb1200_5_90 package since mesh is shared-->
+          <mesh filename="package://abb_irb1200_support/meshes/irb1200_5_90/visual/link_1.dae" scale="0.001 0.001 0.001" />
         </geometry>
         <material name="graphite_white"/>
@@ -45,5 +47,5 @@
       <visual name="visual">
         <geometry>
-          <mesh filename="package://abb_irb1200_support/meshes/irb1200_7_70/visual/link_2.stl" scale="0.001 0.001 0.001" />
+          <mesh filename="package://abb_irb1200_support/meshes/irb1200_7_70/visual/link_2.dae" scale="0.001 0.001 0.001" />
         </geometry>
         <origin xyz="0 0 -0.399" />
@@ -61,5 +63,5 @@
       <visual name="visual">
         <geometry>
-          <mesh filename="package://abb_irb1200_support/meshes/irb1200_7_70/visual/link_3.stl" scale="0.001 0.001 0.001" />
+          <mesh filename="package://abb_irb1200_support/meshes/irb1200_7_70/visual/link_3.dae" scale="0.001 0.001 0.001" />
         </geometry>
         <origin xyz="0 0 -0.749" />
@@ -77,5 +79,6 @@
       <visual name="visual">
         <geometry>
-          <mesh filename="package://abb_irb1200_support/meshes/irb1200_7_70/visual/link_4.stl" scale="0.001 0.001 0.001" />
+	  <!-- reference irb1200_5_90 package since mesh is shared-->
+          <mesh filename="package://abb_irb1200_support/meshes/irb1200_5_90/visual/link_4.dae" scale="0.001 0.001 0.001" />
         </geometry>
         <origin xyz="0 0 ${-0.749 - 0.042}" />
@@ -93,5 +96,6 @@
       <visual name="visual">
         <geometry>
-          <mesh filename="package://abb_irb1200_support/meshes/irb1200_7_70/visual/link_5.stl" scale="0.001 0.001 0.001" />
+	  <!-- reference irb1200_5_90 package since mesh is shared-->
+          <mesh filename="package://abb_irb1200_support/meshes/irb1200_5_90/visual/link_5.dae" scale="0.001 0.001 0.001" />
         </geometry>
         <origin xyz="-0.351 0 ${-0.749 - 0.042}" />
@@ -109,5 +113,6 @@
       <visual name="visual">
         <geometry>
-          <mesh filename="package://abb_irb1200_support/meshes/irb1200_7_70/visual/link_6.stl" scale="0.001 0.001 0.001" />
+	  <!-- reference irb1200_5_90 package since mesh is shared-->
+          <mesh filename="package://abb_irb1200_support/meshes/irb1200_5_90/visual/link_6.dae" scale="0.001 0.001 0.001" />
         </geometry>
         <origin xyz="${-0.351 - 0.082} 0 ${-0.749 - 0.042}" />
